File: kicad/Coffee Timer.sch (KiCad schematic (older format))
At the start: 28 parts, among them J1 Screw_Terminal_01x02, Q1 PN2222A, SW1 SW_Push, SW2 SW_Push, U1 ATtiny85-20PU, U3 74HC595, U4 74HC595

Commit message: fix
Changed lines of the file:
@@
 Text GLabel 6200 6650 2    50   Input ~ 0
 LED_CAT_4
+$Comp
+L power:PWR_FLAG #FLG0101
+U 1 1 5FFF724C
+P 7800 1000
+F 0 "#FLG0101" H 7800 1075 50  0001 C CNN
+F 1 "PWR_FLAG" V 7800 1127 50  0000 L CNN
+F 2 "" H 7800 1000 50  0001 C CNN
+F 3 "~" H 7800 1000 50  0001 C CNN
+	1    7800 1000
+	0    -1   -1   0
+$EndComp
+Connection ~ 7800 1000
+$Comp
+L power:PWR_FLAG #FLG0102
+U 1 1 5FFF7D7F
+P 7800 1100
+F 0 "#FLG0102" H 7800 1175 50  0001 C CNN
+F 1 "PWR_FLAG" V 7800 1227 50  0000 L CNN
+F 2 "" H 7800 1100 50  0001 C CNN
+F 3 "~" H 7800 1100 50  0001 C CNN
+	1    7800 1100
+	0    -1   -1   0
+$EndComp
+Connection ~ 7800 1100
 $EndSCHEMATC
